Commit message: Revert "Merging debug branch to main (#11)"
This reverts commit 0690664276e176c82faa8afb69004c3538b82e7e.

File: urdf/franka_robot.xacro (robot description, xacro)
@@ -9,5 +9,4 @@
     <!-- Is the robot being simulated in gazebo?" -->
     <xacro:arg name="gazebo" default="false" />
-    <xacro:arg name="simulate_camera" default="false" />
     <xacro:include filename="$(find panda_torque_mpc)/urdf/utils.xacro" />
     <xacro:include filename="$(find panda_torque_mpc)/urdf/franka_arm.xacro" />
@@ -67,7 +66,5 @@
       <origin xyz="0 0 0" rpy="3.141592653589793 0 0"/>
     </joint>
-    <xacro:property name="gz_on" value="$(arg gazebo)" />
-    <xacro:property name="sim_cam_on" value="$(arg simulate_camera)" />
-    <xacro:if value="${gz_on and sim_cam_on}">
+    <xacro:if value="$(arg gazebo)">
       <xacro:include filename="$(find panda_torque_mpc)/urdf/_d435.gazebo.xacro"/>
       <xacro:gazebo_d435 camera_name="d435"
