Commit message: Create simple motion capture relay node for the demo

File: urdf/support.urdf.xacro (robot description, xacro)
@@ -45,5 +45,5 @@
         </collision> -->
       </link>
-      <link name="the_ball">
+      <!-- <link name="the_ball">
         <inertial>
           <mass value="1"/>
@@ -66,5 +66,5 @@
           </geometry>
         </collision>
-      </link>
+      </link> -->
       <link name="wall_link_1">
         <inertial>
@@ -206,9 +206,9 @@
         <child link="panda1_box"/>
       </joint>
-      <joint name="the_ball_joint" type="fixed">
+      <!-- <joint name="the_ball_joint" type="fixed">
         <origin xyz="0 0 0.8" />
         <parent link="world"/>
         <child link="the_ball"/>
-      </joint>
+      </joint> -->
   </xacro:macro>
 </robot>
